Commit message: Testing with new big size dae

File: src/g_arm_description/urdf/base.urdf.xacro (robot description, xacro)
@@ -10,3 +10,28 @@
   </visual>
   </link>
+  <!-- Definition of the motors base link -->
+  <link name="motors_link">
+    <visual>
+      <origin rpy="0 0 0" xyz="0 0 0" />
+      <geometry>
+        <mesh filename="package://g_arm_description/meshes/motors.dae"/>
+      </geometry>
+  </visual>
+  </link>
+  <joint name="base_rotation" type="revolute">
+    <origin
+      xyz="0 0 0"
+      rpy="0 0 0" />
+    <parent
+      link="base_link" />
+    <child
+      link="motors_link" />
+    <axis
+      xyz="0 0 1" />
+    <limit
+      lower="0"
+      upper="0"
+      effort="200"
+      velocity="200" />
+  </joint>
 </robot>
