Commit message: URDF easy part done, remains the complex joints

File: src/software/g_arm_description/urdf/base.urdf.xacro (robot description, xacro)
@@ -19,5 +19,23 @@
   </visual>
   </link>
-  <joint name="base_rotation" type="revolute">
+  <!-- Definition of the arm link 1 -->
+  <link name="link1">
+    <visual>
+      <origin rpy="0 0 0" xyz="0 0 0" />
+      <geometry>
+        <mesh filename="package://g_arm_description/meshes/link1.dae"/>
+      </geometry>
+  </visual>
+  </link>
+  <!-- Definition of the arm link 2 -->
+  <link name="link2">
+    <visual>
+      <origin rpy="0 0 0" xyz="0 0 0" />
+      <geometry>
+        <mesh filename="package://g_arm_description/meshes/link2.dae"/>
+      </geometry>
+  </visual>
+  </link>
+  <joint name="joint1" type="revolute">
     <origin
       xyz="0 0 0.076"
@@ -30,8 +48,40 @@
       xyz="0 0 1" />
     <limit
-      lower="0"
-      upper="0"
-      effort="200"
-      velocity="200" />
+      lower="0.0"
+      upper="0.0"
+      effort="200.0"
+      velocity="200.0" />
+  </joint>
+  <joint name="joint2" type="revolute">
+    <origin
+      xyz="0.035 0.0331 0.054"
+      rpy="1.5708 0 0" />
+    <parent
+      link="motors_link" />
+    <child
+      link="link1" />
+    <axis
+      xyz="0 0 1" />
+    <limit
+      lower="0.0"
+      upper="0.0"
+      effort="200.0"
+      velocity="200.0" />
+  </joint>
+  <joint name="joint3" type="revolute">
+    <origin
+      xyz="0.0 0.17 0.0362"
+      rpy="0 0 1.5708" />
+    <parent
+      link="link1" />
+    <child
+      link="link2" />
+    <axis
+      xyz="0 0 1" />
+    <limit
+      lower="0.0"
+      upper="0.0"
+      effort="200.0"
+      velocity="200.0" />
   </joint>
 </robot>

Commit message: Collisions

File: src/software/g_arm_description/urdf/base.urdf.xacro (robot description, xacro)
@@ -8,5 +8,14 @@
         <mesh filename="package://g_arm_description/meshes/base.dae"/>
       </geometry>
-  </visual>
+    </visual>
+    <collision>
+      <origin rpy="0 0 0" xyz="0 0 0.035" />
+      <geometry>
+            <cylinder radius="0.07" length="0.07"/>
+      </geometry>
+      <material name="blue">
+        <color rgba="0 0 1 1"/>
+      </material>
+    </collision>
   </link>
   <!-- Definition of the motors base link -->
@@ -17,5 +26,14 @@
         <mesh filename="package://g_arm_description/meshes/motors.dae"/>
       </geometry>
-  </visual>
+    </visual>
+    <collision>
+      <origin rpy="0 0 0" xyz="-0.00975 0 0.0445" />
+      <geometry>
+            <box size="0.159 0.210 0.089"/> r
+      </geometry>
+      <material name="blue">
+        <color rgba="0 0 1 1"/>
+      </material>
+    </collision>
   </link>
   <!-- Definition of the arm link 1 -->
@@ -26,5 +44,14 @@
         <mesh filename="package://g_arm_description/meshes/link1.dae"/>
       </geometry>
-  </visual>
+    </visual>
+    <collision>
+      <origin rpy="0 0 0" xyz="0.0 0.0975 0.028" />
+      <geometry>
+            <box size="0.035 0.195 0.034"/> r
+      </geometry>
+      <material name="blue">
+        <color rgba="0 0 1 1"/>
+      </material>
+    </collision>
   </link>
   <!-- Definition of the arm link 2 -->
@@ -35,5 +62,14 @@
         <mesh filename="package://g_arm_description/meshes/link2.dae"/>
       </geometry>
-  </visual>
+    </visual>
+    <collision>
+      <origin rpy="0 0 0" xyz="0.0 -0.0675 0.0085" />
+      <geometry>
+            <box size="0.025 0.230 0.015"/> r
+      </geometry>
+      <material name="blue">
+        <color rgba="0 0 1 1"/>
+      </material>
+    </collision>
   </link>
   <joint name="joint1" type="revolute">
@@ -48,6 +84,6 @@
       xyz="0 0 1" />
     <limit
-      lower="0.0"
-      upper="0.0"
+      lower="-1.5707"
+      upper="1.5707"
       effort="200.0"
       velocity="200.0" />
@@ -64,6 +100,6 @@
       xyz="0 0 1" />
     <limit
-      lower="0.0"
-      upper="0.0"
+      lower="-1.5707"
+      upper="1.5707"
       effort="200.0"
       velocity="200.0" />
@@ -80,6 +116,6 @@
       xyz="0 0 1" />
     <limit
-      lower="0.0"
-      upper="0.0"
+      lower="-1.5707"
+      upper="1.5707"
       effort="200.0"
       velocity="200.0" />

Commit message: End-effector mimic

File: src/software/g_arm_description/urdf/base.urdf.xacro (robot description, xacro)
@@ -73,4 +73,25 @@
     </collision>
   </link>
+  <!-- Definition of the arm end effector -->
+  <link name="end_effector">
+    <visual>
+      <origin rpy="0 0 0" xyz="0 0 0" />
+      <geometry>
+        <mesh filename="package://g_arm_description/meshes/end.dae"/>
+      </geometry>
+    </visual>
+    <collision>
+      <origin rpy="0 0 0" xyz="0.0 -0.0675 0.0085" />
+      <geometry>
+            <box size="0.05 0.05 0.05"/> r
+      </geometry>
+      <material name="blue">
+        <color rgba="0 0 1 1"/>
+      </material>
+    </collision>
+  </link>
+    <!-- Definition of the invisible link of the end effector -->
+  <link name="invisible_end">
+  </link>
   <joint name="joint1" type="revolute">
     <origin
@@ -121,3 +142,43 @@
       velocity="200.0" />
   </joint>
+  <joint name="passive_joint4_mimic1" type="revolute">
+    <origin
+      xyz="0.0 -0.17 0.0"
+      rpy="0 0 -1.5708" />
+    <parent
+      link="link2" />
+    <child
+      link="invisible_end" />
+    <axis
+      xyz="0 0 1" />
+    <limit
+      lower="-1.5707"
+      upper="1.5707"
+      effort="200.0"
+      velocity="200.0" />
+    <mimic
+      joint="joint2"
+      multiplier="-1"
+    />
+  </joint>
+  <joint name="passive_joint4_mimic2" type="revolute">
+    <origin
+      xyz="0.0 0.0 0.0"
+      rpy="0 0 0" />
+    <parent
+      link="invisible_end" />
+    <child
+      link="end_effector" />
+    <axis
+      xyz="0 0 1" />
+    <limit
+      lower="-1.5707"
+      upper="1.5707"
+      effort="200.0"
+      velocity="200.0" />
+    <mimic
+      joint="joint3"
+      multiplier="-1"
+    />
+  </joint>
 </robot>

Commit message: Parallelogram 1 done in URDF

File: src/software/g_arm_description/urdf/base.urdf.xacro (robot description, xacro)
@@ -59,5 +59,5 @@
       <origin rpy="0 0 0" xyz="0 0 0" />
       <geometry>
-        <mesh filename="package://g_arm_description/meshes/visual_link_j3_lever.dae"/>
+        <mesh filename="package://g_arm_description/meshes/link_j3_lever.dae"/>
       </geometry>
     </visual>
@@ -216,3 +216,61 @@
     />
   </joint>
+  <!--Rest of the palalegrams: This is not neccesary for the IK but its important for appearance and collision avoidance-->
+  <link name="link_j3_lever_to_rod_intermediate">
+  </link>
+  <link name="link_j3_rod">
+    <visual>
+      <origin rpy="0 0 0" xyz="0 0 0" />
+      <geometry>
+        <mesh filename="package://g_arm_description/meshes/link_j3_rod.dae"/>
+      </geometry>
+    </visual>
+    <collision>
+      <origin rpy="0 0 0" xyz="0.0 -0.0675 0.0085" />
+      <geometry>
+            <box size="0.05 0.05 0.05"/> r
+      </geometry>
+      <material name="blue">
+        <color rgba="0 0 1 1"/>
+      </material>
+    </collision>
+  </link>
+  <joint name="passive_joint_j3_lever_to_rod_intermediate" type="revolute">
+    <origin
+      xyz="-0.035 0.0 -0.030"
+      rpy="0 0 0" />
+    <parent
+      link="link_j3_lever" />
+    <child
+      link="link_j3_lever_to_rod_intermediate" />
+    <axis
+      xyz="0 0 1" />
+    <limit
+      lower="-1.5707"
+      upper="1.5707"
+      effort="200.0"
+      velocity="200.0" />
+    <mimic
+      joint="joint2"
+      multiplier="1"/>
+  </joint>
+  <joint name="passive_joint_j3_lever_to_rod" type="revolute">
+    <origin
+      xyz="0.0 0.0 0.0"
+      rpy="0 0 0" />
+    <parent
+      link="link_j3_lever_to_rod_intermediate" />
+    <child
+      link="link_j3_rod" />
+    <axis
+      xyz="0 0 1" />
+    <limit
+      lower="-1.5707"
+      upper="1.5707"
+      effort="200.0"
+      velocity="200.0" />
+    <mimic
+      joint="joint3"
+      multiplier="-1"/>
+  </joint>
 </robot>

Commit message: Added 2 parts virtuals to urdf

File: src/software/g_arm_description/urdf/base.urdf.xacro (robot description, xacro)
@@ -128,5 +128,5 @@
   <joint name="joint2" type="revolute">
     <origin
-      xyz="0.035 0.0331 0.054"
+      xyz="0.035 0.0331 0.055"
       rpy="1.5708 0 0" />
     <parent
@@ -144,5 +144,5 @@
   <joint name="joint3" type="revolute">
     <origin
-      xyz="0.035 -0.0341 0.054"
+      xyz="0.035 -0.0341 0.055"
       rpy="1.5708 0 0" />
     <parent
@@ -274,3 +274,75 @@
       multiplier="-1"/>
   </joint>
+  <link name="elbow_link">
+    <visual>
+      <origin rpy="0 0 0" xyz="0 0 0" />
+      <geometry>
+        <mesh filename="package://g_arm_description/meshes/elbow.dae"/>
+      </geometry>
+    </visual>
+    <collision>
+      <origin rpy="0 0 0" xyz="0.0 -0.0675 0.0085" />
+      <geometry>
+            <box size="0.05 0.05 0.05"/> r
+      </geometry>
+      <material name="blue">
+        <color rgba="0 0 1 1"/>
+      </material>
+    </collision>
+  </link>
+  <joint name="passive_elbow_joint" type="revolute">
+    <origin
+      xyz="0.0 0.17 0.009"
+      rpy="0 0 0" />
+    <parent
+      link="link1" />
+    <child
+      link="elbow_link" />
+    <axis
+      xyz="0 0 1" />
+    <limit
+      lower="-1.5707"
+      upper="1.5707"
+      effort="200.0"
+      velocity="200.0" />
+    <mimic
+      joint="joint2"
+      multiplier="-1"/>
+  </joint>
+  <link name="parallel_end_link1">
+    <visual>
+      <origin rpy="0 0 0" xyz="0 0 0" />
+      <geometry>
+        <mesh filename="package://g_arm_description/meshes/parallel_end_link1.dae"/>
+      </geometry>
+    </visual>
+    <collision>
+      <origin rpy="0 0 0" xyz="0.0 -0.0675 0.0085" />
+      <geometry>
+            <box size="0.05 0.05 0.05"/> r
+      </geometry>
+      <material name="blue">
+        <color rgba="0 0 1 1"/>
+      </material>
+    </collision>
+  </link>
+  <joint name="passive_parallel_link1_joint" type="revolute">
+    <origin
+      xyz="0.004474 0.058 0.080712"
+      rpy="1.5707 0 0" />
+    <parent
+      link="motors_link" />
+    <child
+      link="parallel_end_link1" />
+    <axis
+      xyz="0 0 1" />
+    <limit
+      lower="-1.5707"
+      upper="1.5707"
+      effort="200.0"
+      velocity="200.0" />
+    <mimic
+      joint="joint2"
+      multiplier="-1"/>
+  </joint>
 </robot>

Commit message: End of the URDF visual

File: src/software/g_arm_description/urdf/base.urdf.xacro (robot description, xacro)
@@ -344,5 +344,41 @@
     <mimic
       joint="joint2"
-      multiplier="-1"/>
+      multiplier="1"/>
+  </joint>
+  <link name="parallel_end_link2">
+    <visual>
+      <origin rpy="0 0 0" xyz="0 0 0" />
+      <geometry>
+        <mesh filename="package://g_arm_description/meshes/parallel_end_link2.dae"/>
+      </geometry>
+    </visual>
+    <collision>
+      <origin rpy="0 0 0" xyz="0.0 -0.0675 0.0085" />
+      <geometry>
+            <box size="0.025 0.230 0.015"/> r
+      </geometry>
+      <material name="blue">
+        <color rgba="0 0 1 1"/>
+      </material>
+    </collision>
+  </link>
+  <joint name="passive_parallel_link2_intermediate" type="revolute">
+    <origin
+      xyz="0.029054 0.019516 -0.011"
+      rpy="0 0 1.5708" />
+    <parent
+      link="elbow_link" />
+    <child
+      link="parallel_end_link2" />
+    <axis
+      xyz="0 0 1" />
+    <limit
+      lower="-1.5707"
+      upper="1.5707"
+      effort="200.0"
+      velocity="200.0" />
+    <mimic
+      joint="joint3"
+      multiplier="1"/>
   </joint>
 </robot>

Commit message: Added precise collisions to URDF

File: src/software/g_arm_description/urdf/base.urdf.xacro (robot description, xacro)
@@ -28,7 +28,7 @@
     </visual>
     <collision>
-      <origin rpy="0 0 0" xyz="-0.00975 0 0.0445" />
-      <geometry>
-            <box size="0.159 0.210 0.089"/> r
+      <origin rpy="0 0 0" xyz="0 0 0" />
+      <geometry>
+          <mesh filename="package://g_arm_description/meshes/motors.stl" scale="0.001 0.001 0.001"/>
       </geometry>
       <material name="blue">
@@ -46,7 +46,7 @@
     </visual>
     <collision>
-      <origin rpy="0 0 0" xyz="0.0 0.0975 0.028" />
-      <geometry>
-            <box size="0.035 0.195 0.034"/> r
+      <origin rpy="0 0 0" xyz="0.0 0.0 0.0" />
+      <geometry>
+        <mesh filename="package://g_arm_description/meshes/link1.stl" scale="0.001 0.001 0.001"/>
       </geometry>
       <material name="blue">
@@ -63,7 +63,7 @@
     </visual>
     <collision>
-      <origin rpy="0 0 0" xyz="0.0 0.0975 0.028" />
-      <geometry>
-            <box size="0.035 0.195 0.034"/> r
+      <origin rpy="0 0 0" xyz="0.0 0.0 0.0" />
+      <geometry>
+        <mesh filename="package://g_arm_description/meshes/link_j3_lever.stl" scale="0.001 0.001 0.001"/>
       </geometry>
       <material name="blue">
@@ -83,7 +83,7 @@
     </visual>
     <collision>
-      <origin rpy="0 0 0" xyz="0.0 -0.0675 0.0085" />
-      <geometry>
-            <box size="0.025 0.230 0.015"/> r
+      <origin rpy="0 0 0" xyz="0.0 0.0 0.0" />
+      <geometry>
+        <mesh filename="package://g_arm_description/meshes/link2.stl" scale="0.001 0.001 0.001"/>
       </geometry>
       <material name="blue">
@@ -101,7 +101,7 @@
     </visual>
     <collision>
-      <origin rpy="0 0 0" xyz="0.0 -0.0675 0.0085" />
-      <geometry>
-            <box size="0.05 0.05 0.05"/> r
+      <origin rpy="0 0 0" xyz="0.0 0.0 0.0" />
+      <geometry>
+        <mesh filename="package://g_arm_description/meshes/end.stl" scale="0.001 0.001 0.001"/>
       </geometry>
       <material name="blue">
@@ -227,7 +227,7 @@
     </visual>
     <collision>
-      <origin rpy="0 0 0" xyz="0.0 -0.0675 0.0085" />
-      <geometry>
-            <box size="0.05 0.05 0.05"/> r
+      <origin rpy="0 0 0" xyz="0.0 0.0 0.0" />
+      <geometry>
+        <mesh filename="package://g_arm_description/meshes/link_j3_rod.stl" scale="0.001 0.001 0.001"/>
       </geometry>
       <material name="blue">
@@ -282,7 +282,7 @@
     </visual>
     <collision>
-      <origin rpy="0 0 0" xyz="0.0 -0.0675 0.0085" />
-      <geometry>
-            <box size="0.05 0.05 0.05"/> r
+      <origin rpy="0 0 0" xyz="0.0 0.0 0.0" />
+      <geometry>
+        <mesh filename="package://g_arm_description/meshes/elbow.stl" scale="0.001 0.001 0.001"/>
       </geometry>
       <material name="blue">
@@ -318,7 +318,7 @@
     </visual>
     <collision>
-      <origin rpy="0 0 0" xyz="0.0 -0.0675 0.0085" />
-      <geometry>
-            <box size="0.05 0.05 0.05"/> r
+      <origin rpy="0 0 0" xyz="0.0 0.0 0.0" />
+      <geometry>
+        <mesh filename="package://g_arm_description/meshes/parallel_end_link1.stl" scale="0.001 0.001 0.001"/>
       </geometry>
       <material name="blue">
@@ -354,7 +354,7 @@
     </visual>
     <collision>
-      <origin rpy="0 0 0" xyz="0.0 -0.0675 0.0085" />
-      <geometry>
-            <box size="0.025 0.230 0.015"/> r
+      <origin rpy="0 0 0" xyz="0.0 0.0 0.0" />
+      <geometry>
+        <mesh filename="package://g_arm_description/meshes/parallel_end_link2.stl" scale="0.001 0.001 0.001"/>
       </geometry>
       <material name="blue">
