Commit message: Fixed start error in moveit package

File: src/software/g_arm_description/urdf/robot.urdf (robot description, URDF)
Before this commit: robot g_arm, 12 links, 11 joints
Joints:
- joint joint1: axis 0 0 1 -> 0.0 0.0 1.0; origin xyz=0 0 0.076 rpy=0 0 0 -> xyz=0.0 0.0 0.076 rpy=0.0 0.0 0.0
- joint joint2: axis 0 0 1 -> 0.0 0.0 1.0
- joint joint3: axis 0 0 1 -> 0.0 0.0 1.0; origin xyz=0.035 -0.0341 0.055 rpy=1.5708 0 0 -> xyz=0.035 -0.0341 0.055 rpy=1.5708 0.0 0.0
- joint joint_link1_link2: axis 0 0 1 -> 0.0 0.0 1.0; mimic joint=joint2 multiplier=-1 -> joint=joint2 multiplier=-1.0
- joint joint_link1_link2_intermediate: axis 0 0 1 -> 0.0 0.0 1.0; mimic joint=joint3 multiplier=1 -> joint=joint3 multiplier=1.0; origin xyz=0.0 0.17 0.0362 rpy=0 0 1.5708 -> xyz=0.0 0.17 0.0362 rpy=0.0 0.0 1.5708
- joint passive_elbow_joint: axis 0 0 1 -> 0.0 0.0 1.0; mimic joint=joint2 multiplier=-1 -> joint=joint2 multiplier=-1.0; origin xyz=0.0 0.17 0.009 rpy=0 0 0 -> xyz=0.0 0.17 0.009 rpy=0.0 0.0 0.0
- joint passive_joint4_mimic: axis 0 0 1 -> 0.0 0.0 1.0; mimic joint=joint3 multiplier=-1 -> joint=joint3 multiplier=-1.0; origin xyz=0.0 -0.17 0.0 rpy=0 0 -1.5708 -> xyz=0.0 -0.17 0.0 rpy=0.0 0.0 -1.5708
- joint passive_joint_j3_lever_to_rod: axis 0 0 1 -> 0.0 0.0 1.0; mimic joint=joint3 multiplier=-1 -> joint=joint3 multiplier=-1.0; origin xyz=0.0 0.0 0.0 rpy=0 0 0 -> xyz=0.0 0.0 0.0 rpy=0.0 0.0 0.0
- joint passive_joint_j3_lever_to_rod_intermediate: axis 0 0 1 -> 0.0 0.0 1.0; mimic joint=joint2 multiplier=1 -> joint=joint2 multiplier=1.0; origin xyz=-0.035 0.0 -0.030 rpy=0 0 0 -> xyz=-0.035 0.0 -0.030 rpy=0.0 0.0 0.0
- joint passive_parallel_link1_joint: axis 0 0 1 -> 0.0 0.0 1.0; mimic joint=joint2 multiplier=1 -> joint=joint2 multiplier=1.0; origin xyz=0.004474 0.058 0.080712 rpy=1.5707 0 0 -> xyz=0.004474 0.058 0.080712 rpy=1.5707 0.0 0.0
- joint passive_parallel_link2_intermediate: axis 0 0 1 -> 0.0 0.0 1.0; mimic joint=joint3 multiplier=1 -> joint=joint3 multiplier=1.0; origin xyz=0.029054 0.019516 -0.011 rpy=0 0 1.5708 -> xyz=0.029054 0.019516 -0.011 rpy=0.0 0.0 1.5708

File: src/software/g_arm_description/urdf/robot.urdf.xacro (robot description, xacro)
@@ -4,5 +4,5 @@
   <link name="base_link">
     <visual>
-      <origin rpy="0 0 0" xyz="0 0 0" />
+      <origin rpy="0.0 0.0 0.0" xyz="0.0 0.0 0.0" />
       <geometry>
         <mesh filename="package://g_arm_description/meshes/base.dae"/>
@@ -10,10 +10,10 @@
     </visual>
     <collision>
-      <origin rpy="0 0 0" xyz="0 0 0.035" />
+      <origin rpy="0.0 0.0 0.0" xyz="0.0 0.0 0.035" />
       <geometry>
             <cylinder radius="0.07" length="0.07"/>
       </geometry>
       <material name="blue">
-        <color rgba="0 0 1 1"/>
+        <color rgba="0.0 0.0 1.0 1.0"/>
       </material>
     </collision>
@@ -22,5 +22,5 @@
   <link name="motors_link">
     <visual>
-      <origin rpy="0 0 0" xyz="0 0 0" />
+      <origin rpy="0.0 0.0 0" xyz="0.0 0.0 0.0" />
       <geometry>
         <mesh filename="package://g_arm_description/meshes/motors.dae"/>
@@ -28,10 +28,10 @@
     </visual>
     <collision>
-      <origin rpy="0 0 0" xyz="0 0 0" />
+      <origin rpy="0.0 0.0 0.0" xyz="0 0 0" />
       <geometry>
           <mesh filename="package://g_arm_description/meshes/motors.stl" scale="0.001 0.001 0.001"/>
       </geometry>
       <material name="blue">
-        <color rgba="0 0 1 1"/>
+        <color rgba="0.0 0.0 1.0 1.0"/>
       </material>
     </collision>
@@ -40,5 +40,5 @@
   <link name="link1">
     <visual>
-      <origin rpy="0 0 0" xyz="0 0 0" />
+      <origin rpy="0.0 0.0 0.0" xyz="0.0 0.0 0.0" />
       <geometry>
         <mesh filename="package://g_arm_description/meshes/link1.dae"/>
@@ -46,10 +46,10 @@
     </visual>
     <collision>
-      <origin rpy="0 0 0" xyz="0.0 0.0 0.0" />
+      <origin rpy="0.0 0.0 0.0" xyz="0.0 0.0 0.0" />
       <geometry>
         <mesh filename="package://g_arm_description/meshes/link1.stl" scale="0.001 0.001 0.001"/>
       </geometry>
       <material name="blue">
-        <color rgba="0 0 1 1"/>
+        <color rgba="0.0 0.0 1.0 1.0"/>
       </material>
     </collision>
@@ -57,5 +57,5 @@
   <link name="link_j3_lever">
     <visual>
-      <origin rpy="0 0 0" xyz="0 0 0" />
+      <origin rpy="0.0 0.0 0.0" xyz="0.0 0.0 0.0" />
       <geometry>
         <mesh filename="package://g_arm_description/meshes/link_j3_lever.dae"/>
@@ -63,10 +63,10 @@
     </visual>
     <collision>
-      <origin rpy="0 0 0" xyz="0.0 0.0 0.0" />
+      <origin rpy="0.0 0.0 0.0" xyz="0.0 0.0 0.0" />
       <geometry>
         <mesh filename="package://g_arm_description/meshes/link_j3_lever.stl" scale="0.001 0.001 0.001"/>
       </geometry>
       <material name="blue">
-        <color rgba="0 0 1 1"/>
+        <color rgba="0.0 0.0 1.0 1.0"/>
       </material>
     </collision>
@@ -77,5 +77,5 @@
   <link name="link2">
     <visual>
-      <origin rpy="0 0 0" xyz="0 0 0" />
+      <origin rpy="0.0 0.0 0.0" xyz="0.0 0.0 0.0" />
       <geometry>
         <mesh filename="package://g_arm_description/meshes/link2.dae"/>
@@ -83,10 +83,10 @@
     </visual>
     <collision>
-      <origin rpy="0 0 0" xyz="0.0 0.0 0.0" />
+      <origin rpy="0.0 0.0 0.0" xyz="0.0 0.0 0.0" />
       <geometry>
         <mesh filename="package://g_arm_description/meshes/link2.stl" scale="0.001 0.001 0.001"/>
       </geometry>
       <material name="blue">
-        <color rgba="0 0 1 1"/>
+        <color rgba="0.0 0.0 1.0 1.0"/>
       </material>
     </collision>
@@ -95,5 +95,5 @@
   <link name="end_effector">
     <visual>
-      <origin rpy="0 0 0" xyz="0 0 0" />
+      <origin rpy="0.0 0.0 0.0" xyz="0.0 0.0 0.0" />
       <geometry>
         <mesh filename="package://g_arm_description/meshes/end.dae"/>
@@ -101,10 +101,10 @@
     </visual>
     <collision>
-      <origin rpy="0 0 0" xyz="0.0 0.0 0.0" />
+      <origin rpy="0.0 0.0 0.0" xyz="0.0 0.0 0.0" />
       <geometry>
         <mesh filename="package://g_arm_description/meshes/end.stl" scale="0.001 0.001 0.001"/>
       </geometry>
       <material name="blue">
-        <color rgba="0 0 1 1"/>
+        <color rgba="0.0 0.0 1.0 1.0"/>
       </material>
     </collision>
@@ -112,6 +112,6 @@
   <joint name="joint1" type="revolute">
     <origin
-      xyz="0 0 0.076"
-      rpy="0 0 0" />
+      xyz="0.0 0.0 0.076"
+      rpy="0.0 0.0 0.0" />
     <parent
       link="base_link" />
@@ -119,5 +119,5 @@
       link="motors_link" />
     <axis
-      xyz="0 0 1" />
+      xyz="0.0 0.0 1.0" />
     <limit
       lower="-1.5707"
@@ -135,5 +135,5 @@
       link="link1" />
     <axis
-      xyz="0 0 1" />
+      xyz="0.0 0.0 1.0" />
     <limit
       lower="-1.5707"
@@ -145,5 +145,5 @@
     <origin
       xyz="0.035 -0.0341 0.055"
-      rpy="1.5708 0 0" />
+      rpy="1.5708 0.0 0.0" />
     <parent
       link="motors_link" />
@@ -151,5 +151,5 @@
       link="link_j3_lever" />
     <axis
-      xyz="0 0 1" />
+      xyz="0.0 0.0 1.0" />
     <limit
       lower="-1.5707"
@@ -161,5 +161,5 @@
     <origin
       xyz="0.0 0.17 0.0362"
-      rpy="0 0 1.5708" />
+      rpy="0.0 0.0 1.5708" />
     <parent
       link="link1" />
@@ -167,5 +167,5 @@
       link="link1_to_link2_intermediate" />
     <axis
-      xyz="0 0 1" />
+      xyz="0.0 0.0 1.0" />
     <limit
       lower="-1.5707"
@@ -175,5 +175,5 @@
     <mimic
       joint="joint3"
-      multiplier="1"/>
+      multiplier="1.0"/>
   </joint>
   <joint name="joint_link1_link2" type="revolute">
@@ -186,5 +186,5 @@
       link="link2" />
     <axis
-      xyz="0 0 1" />
+      xyz="0.0 0.0 1.0" />
     <limit
       lower="-1.5707"
@@ -194,10 +194,10 @@
     <mimic
       joint="joint2"
-      multiplier="-1"/>
+      multiplier="-1.0"/>
   </joint>
   <joint name="passive_joint4_mimic" type="revolute">
     <origin
       xyz="0.0 -0.17 0.0"
-      rpy="0 0 -1.5708" />
+      rpy="0.0 0.0 -1.5708" />
     <parent
       link="link2" />
@@ -205,5 +205,5 @@
       link="end_effector" />
     <axis
-      xyz="0 0 1" />
+      xyz="0.0 0.0 1.0" />
     <limit
       lower="-1.5707"
@@ -213,5 +213,5 @@
     <mimic
       joint="joint3"
-      multiplier="-1"
+      multiplier="-1.0"
     />
   </joint>
@@ -221,5 +221,5 @@
   <link name="link_j3_rod">
     <visual>
-      <origin rpy="0 0 0" xyz="0 0 0" />
+      <origin rpy="0.0 0.0 0.0" xyz="0.0 0.0 0.0" />
       <geometry>
         <mesh filename="package://g_arm_description/meshes/link_j3_rod.dae"/>
@@ -227,10 +227,10 @@
     </visual>
     <collision>
-      <origin rpy="0 0 0" xyz="0.0 0.0 0.0" />
+      <origin rpy="0.0 0.0 0.0" xyz="0.0 0.0 0.0" />
       <geometry>
         <mesh filename="package://g_arm_description/meshes/link_j3_rod.stl" scale="0.001 0.001 0.001"/>
       </geometry>
       <material name="blue">
-        <color rgba="0 0 1 1"/>
+        <color rgba="0.0 0.0 1.0 1.0"/>
       </material>
     </collision>
@@ -239,5 +239,5 @@
     <origin
       xyz="-0.035 0.0 -0.030"
-      rpy="0 0 0" />
+      rpy="0.0 0.0 0.0" />
     <parent
       link="link_j3_lever" />
@@ -245,5 +245,5 @@
       link="link_j3_lever_to_rod_intermediate" />
     <axis
-      xyz="0 0 1" />
+      xyz="0.0 0.0 1.0" />
     <limit
       lower="-1.5707"
@@ -253,10 +253,10 @@
     <mimic
       joint="joint2"
-      multiplier="1"/>
+      multiplier="1.0"/>
   </joint>
   <joint name="passive_joint_j3_lever_to_rod" type="revolute">
     <origin
       xyz="0.0 0.0 0.0"
-      rpy="0 0 0" />
+      rpy="0.0 0.0 0.0" />
     <parent
       link="link_j3_lever_to_rod_intermediate" />
@@ -264,5 +264,5 @@
       link="link_j3_rod" />
     <axis
-      xyz="0 0 1" />
+      xyz="0.0 0.0 1.0" />
     <limit
       lower="-1.5707"
@@ -272,9 +272,9 @@
     <mimic
       joint="joint3"
-      multiplier="-1"/>
+      multiplier="-1.0"/>
   </joint>
   <link name="elbow_link">
     <visual>
-      <origin rpy="0 0 0" xyz="0 0 0" />
+      <origin rpy="0.0 0.0 0.0" xyz="0.0 0.0 0.0" />
       <geometry>
         <mesh filename="package://g_arm_description/meshes/elbow.dae"/>
@@ -282,10 +282,10 @@
     </visual>
     <collision>
-      <origin rpy="0 0 0" xyz="0.0 0.0 0.0" />
+      <origin rpy="0.0 0.0 0.0" xyz="0.0 0.0 0.0" />
       <geometry>
         <mesh filename="package://g_arm_description/meshes/elbow.stl" scale="0.001 0.001 0.001"/>
       </geometry>
       <material name="blue">
-        <color rgba="0 0 1 1"/>
+        <color rgba="0.0 0.0 1.0 1.0"/>
       </material>
     </collision>
@@ -294,5 +294,5 @@
     <origin
       xyz="0.0 0.17 0.009"
-      rpy="0 0 0" />
+      rpy="0.0 0.0 0.0" />
     <parent
       link="link1" />
@@ -300,5 +300,5 @@
       link="elbow_link" />
     <axis
-      xyz="0 0 1" />
+      xyz="0.0 0.0 1.0" />
     <limit
       lower="-1.5707"
@@ -308,9 +308,9 @@
     <mimic
       joint="joint2"
-      multiplier="-1"/>
+      multiplier="-1.0"/>
   </joint>
   <link name="parallel_end_link1">
     <visual>
-      <origin rpy="0 0 0" xyz="0 0 0" />
+      <origin rpy="0.0 0.0 0.0" xyz="0.0 0.0 0.0" />
       <geometry>
         <mesh filename="package://g_arm_description/meshes/parallel_end_link1.dae"/>
@@ -318,10 +318,10 @@
     </visual>
     <collision>
-      <origin rpy="0 0 0" xyz="0.0 0.0 0.0" />
+      <origin rpy="0.0 0.0 0.0" xyz="0.0 0.0 0.0" />
       <geometry>
         <mesh filename="package://g_arm_description/meshes/parallel_end_link1.stl" scale="0.001 0.001 0.001"/>
       </geometry>
       <material name="blue">
-        <color rgba="0 0 1 1"/>
+        <color rgba="0.0 0.0 1.0 1.0"/>
       </material>
     </collision>
@@ -330,5 +330,5 @@
     <origin
       xyz="0.004474 0.058 0.080712"
-      rpy="1.5707 0 0" />
+      rpy="1.5707 0.0 0.0" />
     <parent
       link="motors_link" />
@@ -336,5 +336,5 @@
       link="parallel_end_link1" />
     <axis
-      xyz="0 0 1" />
+      xyz="0.0 0.0 1.0" />
     <limit
       lower="-1.5707"
@@ -344,9 +344,9 @@
     <mimic
       joint="joint2"
-      multiplier="1"/>
+      multiplier="1.0"/>
   </joint>
   <link name="parallel_end_link2">
     <visual>
-      <origin rpy="0 0 0" xyz="0 0 0" />
+      <origin rpy="0.0 0.0 0.0" xyz="0.0 0.0 0.0" />
       <geometry>
         <mesh filename="package://g_arm_description/meshes/parallel_end_link2.dae"/>
@@ -354,10 +354,10 @@
     </visual>
     <collision>
-      <origin rpy="0 0 0" xyz="0.0 0.0 0.0" />
+      <origin rpy="0.0 0.0 0.0" xyz="0.0 0.0 0.0" />
       <geometry>
         <mesh filename="package://g_arm_description/meshes/parallel_end_link2.stl" scale="0.001 0.001 0.001"/>
       </geometry>
       <material name="blue">
-        <color rgba="0 0 1 1"/>
+        <color rgba="0.0 0.0 1.0 1.0"/>
       </material>
     </collision>
@@ -366,5 +366,5 @@
     <origin
       xyz="0.029054 0.019516 -0.011"
-      rpy="0 0 1.5708" />
+      rpy="0.0 0.0 1.5708" />
     <parent
       link="elbow_link" />
@@ -372,5 +372,5 @@
       link="parallel_end_link2" />
     <axis
-      xyz="0 0 1" />
+      xyz="0.0 0.0 1.0" />
     <limit
       lower="-1.5707"
@@ -380,5 +380,5 @@
     <mimic
       joint="joint3"
-      multiplier="1"/>
+      multiplier="1.0"/>
   </joint>
 </robot>

File: src/software/g_arm_moveit/config/g_arm.ros2_control.xacro (robot description, xacro)
@@ -22,11 +22,4 @@
                 <state_interface name="velocity"/>
             </joint>
-            <joint name="joint3">
-                <command_interface name="position"/>
-                <state_interface name="position">
-                  <param name="initial_value">${initial_positions['joint3']}</param>
-                </state_interface>
-                <state_interface name="velocity"/>
-            </joint>
         </ros2_control>
     </xacro:macro>

Commit message: Fixed joint3 overtravel bug

File: src/software/g_arm_description/urdf/robot.urdf (robot description, URDF)
Before this commit: robot g_arm, 12 links, 11 joints
Joints:
- joint joint3: limit lower=-1.5707 upper=1.5707 effort=200.0 velocity=200.0 -> lower=-1.5707 upper=0.1 effort=200.0 velocity=200.0
- joint passive_parallel_link2_intermediate: limit lower=-1.5707 upper=1.5707 effort=200.0 velocity=200.0 -> lower=0.0 upper=0.2 effort=200.0 velocity=200.0

File: src/software/g_arm_description/urdf/robot.urdf.xacro (robot description, xacro)
@@ -154,5 +154,5 @@
     <limit
       lower="-1.5707"
-      upper="1.5707"
+      upper="0.1"
       effort="200.0"
       velocity="200.0" />
@@ -374,6 +374,6 @@
       xyz="0.0 0.0 1.0" />
     <limit
-      lower="-1.5707"
-      upper="1.5707"
+      lower="0.0"
+      upper="0.2"
       effort="200.0"
       velocity="200.0" />

Commit message: Fixed bug not planning because of low range passive link

File: src/software/g_arm_description/urdf/robot.urdf (robot description, URDF)
Before this commit: robot g_arm, 12 links, 11 joints
Joints:
- joint passive_parallel_link2_intermediate: limit lower=0.0 upper=0.2 effort=200.0 velocity=200.0 -> lower=-1.5707 upper=1.5707 effort=200.0 velocity=200.0

File: src/software/g_arm_description/urdf/robot.urdf.xacro (robot description, xacro)
@@ -374,6 +374,6 @@
       xyz="0.0 0.0 1.0" />
     <limit
-      lower="0.0"
-      upper="0.2"
+      lower="-1.5707"
+      upper="1.5707"
       effort="200.0"
       velocity="200.0" />

Commit message: Moveit with Z downwards fixed

File: src/software/g_arm_description/urdf/robot.urdf (robot description, URDF)
Before this commit: robot g_arm, 12 links, 11 joints
Links:
- added link tcp
Joints:
- added joint tcp_joint: type fixed, parent end_effector, child tcp, origin xyz=0.014525 -0.0075 -0.0185 rpy=1.5708 0.0 0.0
- joint passive_parallel_link2_intermediate: limit lower=-1.5707 upper=1.5707 effort=200.0 velocity=200.0 -> lower=-1.5708 upper=1.5708 effort=200.0 velocity=200.0

File: src/software/g_arm_description/urdf/robot.urdf.xacro (robot description, xacro)
@@ -374,6 +374,6 @@
       xyz="0.0 0.0 1.0" />
     <limit
-      lower="-1.5707"
-      upper="1.5707"
+      lower="-1.5708"
+      upper="1.5708"
       effort="200.0"
       velocity="200.0" />
@@ -382,3 +382,14 @@
       multiplier="1.0"/>
   </joint>
+  <link name="tcp">
+  </link>
+  <joint name="tcp_joint" type="fixed">
+    <origin
+      xyz="0.014525 -0.0075 -0.0185"
+      rpy="1.5708 0.0 0.0" />
+    <parent
+      link="end_effector" />
+    <child
+      link="tcp" />
+  </joint>
 </robot>
