Commit message: Working IK

File: src/software/g_arm_description/urdf/robot_electromagnet.urdf (robot description, URDF)
Before this commit: robot g_arm, 15 links, 14 joints
Joints:
- joint joint3: child link_j3_lever -> link1_to_link2_intermediate; limit lower=-1.5707 upper=0.1 effort=200.0 velocity=200.0 -> lower=-1.5707 upper=1.5707 effort=200.0 velocity=200.0; origin xyz=0.035 -0.0341 0.055 rpy=1.5708 0.0 0.0 -> xyz=0.0 0.17 0.0362 rpy=0.0 0.0 1.5708; parent motors_link -> link1
- joint joint_link1_link2_intermediate: child link1_to_link2_intermediate -> link_j3_lever; limit lower=-1.5707 upper=1.5707 effort=200.0 velocity=200.0 -> lower=-1.5707 upper=0.1 effort=200.0 velocity=200.0; origin xyz=0.0 0.17 0.0362 rpy=0.0 0.0 1.5708 -> xyz=0.035 -0.0341 0.055 rpy=1.5708 0.0 0.0; parent link1 -> motors_link

File: src/software/g_arm_description/urdf/robot_electromagnet.urdf.xacro (robot description, xacro)
@@ -142,5 +142,5 @@
       velocity="200.0" />
   </joint>
-  <joint name="joint3" type="revolute">
+  <joint name="joint_link1_link2_intermediate" type="revolute">
     <origin
       xyz="0.035 -0.0341 0.055"
@@ -157,6 +157,9 @@
       effort="200.0"
       velocity="200.0" />
-  </joint>
-  <joint name="joint_link1_link2_intermediate" type="revolute">
+    <mimic
+      joint="joint3"
+      multiplier="1.0"/>
+  </joint>
+  <joint name="joint3" type="revolute">
     <origin
       xyz="0.0 0.17 0.0362"
@@ -173,7 +176,4 @@
       effort="200.0"
       velocity="200.0" />
-    <mimic
-      joint="joint3"
-      multiplier="1.0"/>
   </joint>
   <joint name="joint_link1_link2" type="revolute">

Commit message: Added electromagnet test and works

File: src/software/g_arm_description/urdf/robot_electromagnet.urdf (robot description, URDF)
Before this commit: robot g_arm, 15 links, 14 joints
Joints:
- joint jointPWM: limit lower=0.0 upper=0.001 effort=200.0 velocity=200.0 -> lower=0.0 upper=1.0 effort=200.0 velocity=200.0

File: src/software/g_arm_description/urdf/robot_electromagnet.urdf.xacro (robot description, xacro)
@@ -422,5 +422,5 @@
     <limit
       lower="0.0"
-      upper="0.001"
+      upper="1.0"
       effort="200.0"
       velocity="200.0" />
