Commit message: Launcher of moveit real

File: src/software/g_arm_moveit/config/g_arm.ros2_control.xacro (robot description, xacro)
@@ -22,4 +22,11 @@
                 <state_interface name="velocity"/>
             </joint>
+            <joint name="joint3">
+                <command_interface name="position"/>
+                <state_interface name="position">
+                  <param name="initial_value">${initial_positions['joint3']}</param>
+                </state_interface>
+                <state_interface name="velocity"/>
+            </joint>
         </ros2_control>
     </xacro:macro>
